File: wiring_diagram.kicad_sch (KiCad schematic)
At the start: 9 parts

Commit message: Add files via upload
Parts:
- removed BT1, BT2, BT7, BT9: Battery_Cell, symbol Device:Battery_Cell
Other:
- note added: "Recovery Beacon"
- note removed: "2S 18650"
- note removed: "30cm"
- note removed: "AMP Speed Bridge"
- note removed: "EM_BAT"
- note removed: "FW_BAT"
- note removed: "FW_PWR"
- note removed: "Gray: Featherweight GPS Power (REMOVED)"
- note removed: "VL_BAT"
- note removed: "VL_PYRO_MAIN"
