File: UPDATED_AMP_FINAL.kicad_sch (KiCad schematic)
At the start: 5 parts

Commit message: Add files via upload
Other:
- note added: "GRYPHON"
- note removed: "10cm"
- note removed: "5cm"
- note removed: "ICARUS V2"
