File: UPDATED_AMP_FINAL.kicad_sch (KiCad schematic)
At the start: 24 parts, among them SW1 SW_SPST, SW2 SW_SPST, SW3 SW_SPST, SW4 SW_SPST

Commit message: changes to format
Parts:
- removed R1, R2, R5, R6: E-Match, symbol Device:R_US
- added R3, R4, R5, R6: R, symbol Device:R
Other:
- note added: "E-Matches"
- note added: "E-fuses (7A), 1-4"
- note added: "Mini A.M.P"
- note added: "Screw Switch"
- note removed: "MINI A.M.P"

Commit message: exported PDF
Parts:
- removed E-Fuse(1-4)(7A), E-Fuse3: Fuse, symbol Device:Fuse
- removed F6, F7: Fuse (7A, symbol Device:Fuse
- removed SW3: SW_SPST, symbol Switch:SW_SPST
- added E-Fuse4: Fuse, symbol Device:Fuse
- added F1, F2: Fuse (7A, symbol Device:Fuse
- added SW5: SW_SPST, symbol Switch:SW_SPST
Other:
- note added: "Avionics Bay"
- note added: "Fuse (7A)"
- note added: "Nosecone"

Commit message: updated wiring diagram text (exported updated PDF)
Other:
- note added: "Magnetic Switch"

Commit message: minor changes
Other:
- note added: "E-fuses (7A), 1-3"
- note removed: "E-fuses (7A), 1-4"
- note removed: "Green: EasyMini Power"

Commit message: fixed minor visual errors
Parts:
- removed BT22, BT23: Battery_Cell, symbol Device:Battery_Cell
Other:
- note added: "E-fuse (7A)"
- note removed: "E-fuses (7A), 1-3"
- title: Titan Avionics Bay Wiring Diagram -> Osiris Avionics Bay Wiring Diagram
Changed lines of the file:
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@@
 	(paper "User" 546.1 889)
 	(title_block
-		(title "Titan Avionics Bay Wiring Diagram")
+		(title "Osiris Avionics Bay Wiring Diagram")
 		(date "2026-01-25")
 		(rev "r3")

Commit message: updates to match new layout diagram (wip)
Other:
- note added: "EasyMini"
