File: _autosave-UPDATED_AMP_FINAL.kicad_sch (KiCad schematic)
At the start: 24 parts, among them SW1 SW_SPST, SW2 SW_SPST, SW3 SW_SPST, SW4 SW_SPST

Commit message: changes 2
Other:
- note added: "E-fuses (7A), 1-4"
- note removed: "1.2x3"
