File: FINAL_OSIRIS_WIRING_DIAGRAM.kicad_sch (KiCad schematic)
At the start: 21 parts, among them SW1 SW_SPST, SW2 SW_SPST, SW4 SW_SPST, SW5 SW_SPST

Commit message: Replace old wiring diagram files
Other:
- note added: "BR_PYRO_DORG"
- note added: "CAN_BUS"
- note added: "FW_PWR"
- note added: "GRYPHON"
- note added: "VLF5"
- note removed: "EasyMini"
- note removed: "Gryphon"
