File: Osiris_Wiring_Diagram_July292026.kicad_sch (KiCad schematic)
At the start: 21 parts, among them SW1 SW_SPST, SW2 SW_SPST, SW4 SW_SPST, SW5 SW_SPST

Commit message: VL and BR swap
Other:
- note removed: "BR_PYRO_DORG"
